File: Electrical/Board Design/_autosave-clock.kicad_pcb (KiCad board)
At the start: 2 copper layers, 133.3 x 50.8 mm, 40 parts, among them CON1 AVR-ISP-6, IC1 ATTINY84A-SS, Q1 FET_N, Q2 FET_P, SW1 SPST, U1 MCP1624, X1 CRYSTAL 32.768kHz

Commit message: checking board layout against knob parts
Parts:
- R2: value 50K -> POTENTIOMETER
Changed lines of the file:
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@@
   (module bourns_knob (layer F.Cu)
     (at 142.875 186.695004 180)
-    (fp_text reference R2 (at -9.5 -0.5 180) (layer F.SilkS)
+    (fp_text reference R2 (at -7.075 -4.28 180) (layer F.SilkS)
       (effects (font (size 1 1) (thickness 0.15)))
     )
-    (fp_text value 50K (at 10 -0.5 180) (layer F.SilkS)
+    (fp_text value POTENTIOMETER (at 2.325 -4.28 180) (layer F.SilkS)
       (effects (font (size 1 1) (thickness 0.15)))
     )
