File: Electrical/Board Design/clock.kicad_pcb (KiCad board)
At the start: 2 copper layers, 133.3 x 50.8 mm, 60 parts, among them CON1 AVR-ISP-6, CON2 USB-MICRO-B, IC1 ATTINY84A-SS, P1 CONN_6, P2 CONN_2, P3 CONN_2, P4 CONN_2, P5 CONN_2, P6 CONN_2, P7 CONN_2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

Commit message: finalized changes and sent to fab
Parts:
- removed BT3, BT4: BATTERY_CLIP, AA_Battery_Clip_THRU_HOLE_BK-92
- added BREAK_TAB: Val**, BREAK_HOLE, F.Cu at (63.2, 119.3)
- added BREAK_TAB: Val**, BREAK_HOLE, F.Cu at (58.9, 119.3)
- added BREAK_TAB: Val**, BREAK_HOLE, F.Cu at (60.7, 119.3)
- added P9: CONN_2, TE-connectivity-2, F.Cu at (125.7, 121.0)
- P8: value CONN_2 -> SPKR
- moved SW1 67.5 mm to (125.7, 111.0), turned to 180 degrees
- moved R3 14.4 mm to (64.8, 86.4)
- moved P8 9.93 mm to (136.3, 121.3)
- moved D4 9.92 mm to (140.7, 111.6)
- moved P7 9.92 mm to (145.8, 121.2)
- moved Q5 9.92 mm to (149.0, 112.3)
- moved R13 9.92 mm to (143.9, 111.6)
- moved D1 9.91 mm to (136.3, 116.0)
- moved R15 6.23 mm to (163.1, 110.7)
- moved D3 6.23 mm to (154.8, 120.9)
- moved P5 6.23 mm to (164.3, 120.9)
- moved Q3 6.23 mm to (168.8, 112.0)
- moved P4 2.91 mm to (81.0, 121.7)
- moved C9 2.87 mm to (60.3, 122.2)
Connections:
- P5 pad 1: N-0000029 (its old number) -> +5V
- R15 pad 1: N-0000029 (its old number) -> +5V
Routing:
- net +5V: track 62.5 -> 216.7 mm, vias 0 -> 4
- net VCC: track 14.1 -> 163.8 mm, vias 0 -> 9
- net /BATTERY POWER: track 52.8 -> 155.3 mm, vias 3 -> 7
- net N-0000015: track 8.37 -> 89.2 mm, vias 0 -> 7
- net /MODE SELECT POWER: track 34.8 -> 92.3 mm
- net GND: track 41.3 -> 57.1 mm, vias 10 -> 18
- net N-0000029 (its old number): track 5.34 -> 0.00 mm
- net /HOURS: track 82.6 -> 87.6 mm
- net /ALARM BUZZER: track 114.7 -> 110.0 mm, vias 6 -> 3
- net /AM PM LIGHT: track 113.7 -> 118.1 mm, vias 6 -> 4
- net N-0000016: track 10.2 -> 13.4 mm
- net N-0000014: track 58.1 -> 56.1 mm
- net /MODE SELECT: track 75.3 -> 73.8 mm
- net /INT 2: track 21.1 -> 20.6 mm
Other:
- outline, holes or cut-outs redrawn
- board text added: "SWITCH"
- board text added: "awkwardengineer.com"
- board text added: "for help, send email to questions@awkwardengineer.com"
- board text removed: "www.awkwardengineer.com"
